Commit message: Gripper Position 0.04 => 0.00

File: urdf_ur5_ur3_gripper/ur3_robotiq85_gripper.urdf.xacro (robot description, xacro)
@@ -30,5 +30,5 @@
   <!-- Robotiq Coupler Joint an tool0-Link -->
   <joint name="robotiq_coupler_joint" type="fixed">
-    <origin xyz="0 0 0.04" rpy="0 0 ${-pi/2.0}" />
+    <origin xyz="0 0 0.0" rpy="0 0 ${-pi/2.0}" />
     <parent link="tool0"/>
     <child link="robotiq_coupler"/>
